Commit message: added camera branch and corrected direction of motion

File: urdf/test_diff_drive.xacro.urdf (robot description, URDF)
Before this commit: robot diff_drive, 4 links, 3 joints
Links:
- added link camera_link, mass 0.1; collision box size=0.1 0.1 0.1; visual box size=0.1 0.1 0.1
Joints:
- added joint camera_joint: type fixed, parent chassis, child camera_link, origin xyz=0 0 1.0 rpy=0 0 0
- joint caster_joint: origin xyz=-0.957138 -0 0.2 rpy=0 0 0 -> xyz=0.55 0 0.2 rpy=0 0 0
- joint left_wheel_joint: axis 0 0 1 -> 0 1 0; origin xyz=0.554283 0.625029 0.3 rpy=-1.5707 0 0 -> xyz=-0.95 0.625029 0.3 rpy=0 0 0
- joint right_wheel_joint: axis 0 0 1 -> 0 1 0; origin xyz=0.554283 -0.625029 0.3 rpy=-1.5707 0 0 -> xyz=-0.95 -0.625029 0.3 rpy=0 0 0

Commit message: corrected direction of motion

File: urdf/test_diff_drive.xacro.urdf (robot description, URDF)
Before this commit: robot diff_drive, 4 links, 3 joints
Joints:
- joint caster_joint: origin xyz=-0.957138 -0 0.2 rpy=0 0 0 -> xyz=0.55 0 0.2 rpy=0 0 0
- joint left_wheel_joint: axis 0 0 1 -> 0 1 0; origin xyz=0.554283 0.625029 0.3 rpy=-1.5707 0 0 -> xyz=-0.95 0.625029 0.3 rpy=0 0 0
- joint right_wheel_joint: axis 0 0 1 -> 0 1 0; origin xyz=0.554283 -0.625029 0.3 rpy=-1.5707 0 0 -> xyz=-0.95 -0.625029 0.3 rpy=0 0 0
